Commit message: urdf of robot

File: src/robot_describe/urdf/xacro/robot.xacro (robot description, xacro)
@@ -1,3 +1,4 @@
 <robot xmlns:xacro="http://www.ros.org/wiki/xacro" name="inverted_pendulum">
+    <xacro:property name="PI" value="3.1415"/>
     <!-- base_link -->
     <xacro:property name="base_length" value="1"/>
@@ -22,3 +23,64 @@
         <origin xyz="0.0 0.0 ${base_height / 2}" rpy="0.0 0.0 0.0"/>
     </joint>
+    <!-- sliding block -->
+    <xacro:property name="block_length" value="${base_width}"/>
+    <xacro:property name="block_width" value="${base_width}"/>
+    <xacro:property name="block_height" value="${base_width}"/>
+    <link name="sliding_block">
+        <visual>
+            <origin xyz="0.0 0.0 ${block_height/2}" rpy="0.0 0.0 0.0"/>
+            <geometry>
+                <box size="${block_length} ${block_width} ${block_height}"/>
+            </geometry>
+            <material name="red">
+                <color rgba="1.0 0.0 0.0 1"/>
+            </material>
+        </visual>
+    </link>
+    <joint name="s_block2base" type="prismatic">
+        <origin xyz="${(base_length - block_length)/2} 0.0 ${base_height/2}" rpy="0.0 0.0 0.0"/>
+        <parent link="base"/>
+        <child link="sliding_block"/>
+        <axis xyz="-1 0.0 0.0"/>
+        <limit lower="0.0" upper="${base_length - block_length}" effort="2" velocity="0.5"/>
+    </joint>
+    <!-- rotating block -->
+    <xacro:property name="r_block_radius" value="0.005"/>
+    <xacro:property name="r_block_length" value="0.01"/>
+    <link name="rotating_block">
+        <visual>
+            <origin xyz="0 ${(r_block_length+block_width)/2} 0.0" rpy="${PI/2} 0.0 0.0"/>
+            <geometry>
+                <cylinder radius="${r_block_radius}" length="${r_block_length}"/>
+            </geometry>
+            <material name="white">
+                <color rgba="1.0 1.0 1.0 1"/>
+            </material>
+        </visual>
+    </link>
+    <joint name="r_block2s_block" type="continuous">
+        <parent link="sliding_block"/>
+        <child link="rotating_block"/>
+        <origin xyz="0.0 0.0 ${block_height/2}" rpy="0.0 0.0 0.0"/>
+        <axis xyz="0.0 1 0.0"/>
+    </joint>
+    <!-- rod -->
+    <xacro:property name="rod_radius" value="0.0025"/>
+    <xacro:property name="rod_length" value="${(base_height+block_height)/2}"/>
+    <link name="rod">
+        <visual>
+            <origin xyz="0 ${base_width/2+rod_radius+r_block_length/2} ${-1*rod_length/2}" rpy="0.0 0.0 0.0"/>
+            <geometry>
+                <cylinder radius="${rod_radius}" length="${rod_length}"/>
+            </geometry>
+            <material name="green">
+                <color rgba="0.0 1.0 0.0 1"/>
+            </material>
+        </visual>
+    </link>
+    <joint name="rod2r_block" type="fixed">
+        <parent link="rotating_block"/>
+        <child link="rod"/>
+        <origin xyz="0.0 0.0 0" rpy="0.0 0.0 0.0"/>
+    </joint>
 </robot>

Commit message: urdf of  gazebo

File: src/robot_describe/urdf/xacro/robot.xacro (robot description, xacro)
@@ -1,3 +1,4 @@
 <robot xmlns:xacro="http://www.ros.org/wiki/xacro" name="inverted_pendulum">
+    <xacro:include filename="calulator.xacro"/>
     <xacro:property name="PI" value="3.1415"/>
     <!-- base_link -->
@@ -5,4 +6,5 @@
     <xacro:property name="base_width" value="0.1"/>
     <xacro:property name="base_height" value="0.5"/>
+    <xacro:property name="base_mass" value="10"/>
     <link name="world">
     </link>
@@ -17,5 +19,17 @@
             </material>
         </visual>
+        <collision>
+            <origin xyz="0.0 0.0 0" rpy="0.0 0.0 0.0"/>
+            <geometry>
+                <box size="${base_length} ${base_width} ${base_height}"/>
+            </geometry>
+        </collision>
+        <xacro:box_inertial_matrix m="${base_mass}" l="${base_length}" w="${base_width}" h="${base_height}"/>
     </link>
+    <gazebo reference="base">
+        <material>
+            Gazebo/Blue
+        </material>
+    </gazebo>
     <joint name="base2world" type="fixed">
         <parent link="world"/>
@@ -27,4 +41,5 @@
     <xacro:property name="block_width" value="${base_width}"/>
     <xacro:property name="block_height" value="${base_width}"/>
+    <xacro:property name="block_mass" value="0.4"/>
     <link name="sliding_block">
         <visual>
@@ -37,5 +52,17 @@
             </material>
         </visual>
+        <collision>
+            <origin xyz="0.0 0.0 ${block_height/2}" rpy="0.0 0.0 0.0"/>
+            <geometry>
+                <box size="${block_length} ${block_width} ${block_height}"/>
+            </geometry>
+        </collision>
+        <xacro:box_inertial_matrix m="${block_mass}" l="${block_length}" w="${block_width}" h="${block_height}"/>
     </link>
+    <gazebo reference="sliding_block">
+        <material>
+            Gazebo/Red
+        </material>
+    </gazebo>
     <joint name="s_block2base" type="prismatic">
         <origin xyz="${(base_length - block_length)/2} 0.0 ${base_height/2}" rpy="0.0 0.0 0.0"/>
@@ -48,4 +75,5 @@
     <xacro:property name="r_block_radius" value="0.005"/>
     <xacro:property name="r_block_length" value="0.01"/>
+    <xacro:property name="r_block_mass" value="0.05"/>
     <link name="rotating_block">
         <visual>
@@ -58,5 +86,17 @@
             </material>
         </visual>
+        <collision>
+            <origin xyz="0 ${(r_block_length+block_width)/2} 0.0" rpy="${PI/2} 0.0 0.0"/>
+            <geometry>
+                <cylinder radius="${r_block_radius}" length="${r_block_length}"/>
+            </geometry>
+        </collision>
+        <xacro:cylinder_inertial_matrix m="${r_block_mass}" r="${r_block_radius}" h="${r_block_length}"/>
     </link>
+    <gazebo reference="rotating_block">
+        <material>
+            Gazebo/White
+        </material>
+    </gazebo>
     <joint name="r_block2s_block" type="continuous">
         <parent link="sliding_block"/>
@@ -68,4 +108,5 @@
     <xacro:property name="rod_radius" value="0.0025"/>
     <xacro:property name="rod_length" value="${(base_height+block_height)/2}"/>
+    <xacro:property name="rod_mass" value="0.4"/>
     <link name="rod">
         <visual>
@@ -78,5 +119,17 @@
             </material>
         </visual>
+        <collision>
+            <origin xyz="0 ${base_width/2+rod_radius+r_block_length/2} ${-1*rod_length/2}" rpy="0.0 0.0 0.0"/>
+            <geometry>
+                <cylinder radius="${rod_radius}" length="${rod_length}"/>
+            </geometry>
+        </collision>
+        <xacro:cylinder_inertial_matrix m="${rod_mass}" r="${rod_radius}" h="${rod_length}"/>
     </link>
+    <gazebo reference="rod">
+        <material>
+            Gazebo/Green
+        </material>
+    </gazebo>
     <joint name="rod2r_block" type="fixed">
         <parent link="rotating_block"/>

Commit message: add controller

File: src/robot_describe/urdf/xacro/robot.xacro (robot description, xacro)
@@ -72,4 +72,19 @@
         <limit lower="0.0" upper="${base_length - block_length}" effort="2" velocity="0.5"/>
     </joint>
+    <transmission name="tran1">
+        <type>transmission_interface/SimpleTransmission</type>
+        <joint name="s_block2base">
+            <hardwareInterface>VelocityJointInterface</hardwareInterface>
+        </joint>
+        <actuator name="motor1">
+            <hardwareInterface>VelocityJointInterface</hardwareInterface>
+            <mechanicalReduction>1</mechanicalReduction>
+        </actuator>
+    </transmission>
+    <gazebo>
+        <plugin name="gazebo_ros_control" filename="libgazebo_ros_control.so">
+        <robotNamespace>/inverted_pendulum</robotNamespace>
+        </plugin>
+    </gazebo>
     <!-- rotating block -->
     <xacro:property name="r_block_radius" value="0.005"/>
@@ -105,4 +120,14 @@
         <axis xyz="0.0 1 0.0"/>
     </joint>
+    <transmission name="tran2">
+        <type>transmission_interface/SimpleTransmission</type>
+        <joint name="r_block2s_block">
+            <hardwareInterface>PositionJointInterface</hardwareInterface>
+        </joint>
+        <actuator name="motor2">
+            <hardwareInterface>PositionJointInterface</hardwareInterface>
+            <mechanicalReduction>1</mechanicalReduction>
+        </actuator>
+    </transmission>
     <!-- rod -->
     <xacro:property name="rod_radius" value="0.0025"/>

Commit message: feat: add controller and transmission

File: src/robot_describe/urdf/xacro/robot.xacro (robot description, xacro)
@@ -41,8 +41,8 @@
     <xacro:property name="block_width" value="${base_width}"/>
     <xacro:property name="block_height" value="${base_width}"/>
-    <xacro:property name="block_mass" value="0.4"/>
+    <xacro:property name="block_mass" value="0.5"/>
     <link name="sliding_block">
         <visual>
-            <origin xyz="0.0 0.0 ${block_height/2}" rpy="0.0 0.0 0.0"/>
+            <origin xyz="0.0 0.0 0" rpy="0.0 0.0 0.0"/>
             <geometry>
                 <box size="${block_length} ${block_width} ${block_height}"/>
@@ -53,5 +53,5 @@
         </visual>
         <collision>
-            <origin xyz="0.0 0.0 ${block_height/2}" rpy="0.0 0.0 0.0"/>
+            <origin xyz="0.0 0.0 0" rpy="0.0 0.0 0.0"/>
             <geometry>
                 <box size="${block_length} ${block_width} ${block_height}"/>
@@ -61,4 +61,6 @@
     </link>
     <gazebo reference="sliding_block">
+        <mu1>0.2</mu1>
+        <mu2>0.2</mu2>
         <material>
             Gazebo/Red
@@ -66,17 +68,19 @@
     </gazebo>
     <joint name="s_block2base" type="prismatic">
-        <origin xyz="${(base_length - block_length)/2} 0.0 ${base_height/2}" rpy="0.0 0.0 0.0"/>
+        <!-- <origin xyz="${(base_length - block_length)/2} 0.0 ${(base_height+block_height)/2}" rpy="0.0 0.0 0.0"/> -->
+        <origin xyz="0 0.0 ${(base_height+block_height)/2}" rpy="0.0 0.0 0.0"/>
         <parent link="base"/>
         <child link="sliding_block"/>
-        <axis xyz="-1 0.0 0.0"/>
-        <limit lower="0.0" upper="${base_length - block_length}" effort="2" velocity="0.5"/>
+        <axis xyz="1 0.0 0.0"/>
+        <limit lower="${-(base_length - block_length)/2}" upper="${(base_length - block_length)/2}" effort="1000" velocity="100"/>
+        <dynamics damping="0.7"/>
     </joint>
     <transmission name="tran1">
         <type>transmission_interface/SimpleTransmission</type>
         <joint name="s_block2base">
-            <hardwareInterface>VelocityJointInterface</hardwareInterface>
+            <hardwareInterface>hardware_interface/EffortJointInterface</hardwareInterface>
         </joint>
         <actuator name="motor1">
-            <hardwareInterface>VelocityJointInterface</hardwareInterface>
+            <hardwareInterface>hardware_interface/EffortJointInterface</hardwareInterface>
             <mechanicalReduction>1</mechanicalReduction>
         </actuator>
@@ -85,4 +89,5 @@
         <plugin name="gazebo_ros_control" filename="libgazebo_ros_control.so">
         <robotNamespace>/inverted_pendulum</robotNamespace>
+        <robotSimType>gazebo_ros_control/DefaultRobotHWSim</robotSimType>
         </plugin>
     </gazebo>
@@ -90,8 +95,8 @@
     <xacro:property name="r_block_radius" value="0.005"/>
     <xacro:property name="r_block_length" value="0.01"/>
-    <xacro:property name="r_block_mass" value="0.05"/>
+    <xacro:property name="r_block_mass" value="0.001"/>
     <link name="rotating_block">
         <visual>
-            <origin xyz="0 ${(r_block_length+block_width)/2} 0.0" rpy="${PI/2} 0.0 0.0"/>
+            <origin xyz="0 0 0.0" rpy="${PI/2} 0.0 0.0"/>
             <geometry>
                 <cylinder radius="${r_block_radius}" length="${r_block_length}"/>
@@ -102,5 +107,5 @@
         </visual>
         <collision>
-            <origin xyz="0 ${(r_block_length+block_width)/2} 0.0" rpy="${PI/2} 0.0 0.0"/>
+            <origin xyz="0 0 0.0" rpy="${PI/2} 0.0 0.0"/>
             <geometry>
                 <cylinder radius="${r_block_radius}" length="${r_block_length}"/>
@@ -110,31 +115,22 @@
     </link>
     <gazebo reference="rotating_block">
+        <mu1>0.2</mu1>
+        <mu2>0.2</mu2>
         <material>
             Gazebo/White
         </material>
     </gazebo>
-    <joint name="r_block2s_block" type="continuous">
+    <joint name="r_block2s_block" type="fixed">
         <parent link="sliding_block"/>
         <child link="rotating_block"/>
-        <origin xyz="0.0 0.0 ${block_height/2}" rpy="0.0 0.0 0.0"/>
-        <axis xyz="0.0 1 0.0"/>
+        <origin xyz="0.0 ${(block_width+r_block_length)/2} 0" rpy="0.0 0.0 0.0"/>
     </joint>
-    <transmission name="tran2">
-        <type>transmission_interface/SimpleTransmission</type>
-        <joint name="r_block2s_block">
-            <hardwareInterface>PositionJointInterface</hardwareInterface>
-        </joint>
-        <actuator name="motor2">
-            <hardwareInterface>PositionJointInterface</hardwareInterface>
-            <mechanicalReduction>1</mechanicalReduction>
-        </actuator>
-    </transmission>
     <!-- rod -->
     <xacro:property name="rod_radius" value="0.0025"/>
     <xacro:property name="rod_length" value="${(base_height+block_height)/2}"/>
-    <xacro:property name="rod_mass" value="0.4"/>
+    <xacro:property name="rod_mass" value="0.2"/>
     <link name="rod">
         <visual>
-            <origin xyz="0 ${base_width/2+rod_radius+r_block_length/2} ${-1*rod_length/2}" rpy="0.0 0.0 0.0"/>
+            <origin xyz="0 0 ${rod_length/2}" rpy="0.0 0.0 0.0"/>
             <geometry>
                 <cylinder radius="${rod_radius}" length="${rod_length}"/>
@@ -145,20 +141,43 @@
         </visual>
         <collision>
-            <origin xyz="0 ${base_width/2+rod_radius+r_block_length/2} ${-1*rod_length/2}" rpy="0.0 0.0 0.0"/>
+            <origin xyz="0 0 ${rod_length/2}" rpy="0.0 0.0 0.0"/>
             <geometry>
                 <cylinder radius="${rod_radius}" length="${rod_length}"/>
             </geometry>
         </collision>
-        <xacro:cylinder_inertial_matrix m="${rod_mass}" r="${rod_radius}" h="${rod_length}"/>
+        <!-- <xacro:cylinder_inertial_matrix m="${rod_mass}" r="${rod_radius}" h="${rod_length}"/> -->
+        <inertial>
+            <mass value="${rod_mass}" />
+            <inertia ixx="${rod_mass*(3*rod_radius*rod_radius+rod_length*rod_length)/12}" ixy = "0" ixz = "0"
+                iyy="${rod_mass*(3*rod_radius*rod_radius+rod_length*rod_length)/12}" iyz = "0"
+                izz="${rod_mass*rod_radius*rod_radius/2}" />
+            <origin xyz="0.0 0.0 ${rod_length/2}" rpy="0.0 0.0 0.0"/>
+        </inertial>
     </link>
     <gazebo reference="rod">
+        <mu1>0.1</mu1>
+        <mu2>0.1</mu2>
         <material>
             Gazebo/Green
         </material>
+        <turnGravityOff>false</turnGravityOff>
     </gazebo>
-    <joint name="rod2r_block" type="fixed">
+    <joint name="rod2r_block" type="continuous">
         <parent link="rotating_block"/>
         <child link="rod"/>
-        <origin xyz="0.0 0.0 0" rpy="0.0 0.0 0.0"/>
+        <origin xyz="0.0 ${rod_radius+r_block_length/2} 0" rpy="0.0 0.0 0.0"/>
+        <axis xyz="0.0 1 0.0"/>
+        <dynamics  damping="0.005"/>
+        <!-- damping="0.02" -->
     </joint>
+    <transmission name="tran2">
+        <type>transmission_interface/SimpleTransmission</type>
+        <joint name="rod2r_block">
+            <hardwareInterface>hardware_interface/EffortJointInterface</hardwareInterface>
+        </joint>
+        <actuator name="motor2">
+            <hardwareInterface>hardware_interface/EffortJointInterface</hardwareInterface>
+            <mechanicalReduction>1</mechanicalReduction>
+        </actuator>
+    </transmission>
 </robot>
